File: KiCad/windemere-basic.kicad_pcb (KiCad board)
At the start: 2 copper layers, 152.4 x 158.7 mm, 65 parts, among them J1 Barrel_Jack, J2 Connector, SW1 Reset Button, U1 L7805, U2 74HC00, U3 WD65C02, U4 28C256, U5 62256, U6 WD65C22, U7 MM74C922, U8 HD44780U, U9 MCP102-475, X1 1MHz

Commit message: update symbols
Parts:
- renumbered J1 to J2, J2 to J3
Changed lines of the file:
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@@
   (net 35 "/A11")
   (net 36 "Net-(D2-Pad1)")
-  (net 37 "Net-(J2-Pad26)")
-  (net 38 "Net-(J2-Pad28)")
-  (net 39 "Net-(J2-Pad30)")
-  (net 40 "Net-(J2-Pad34)")
+  (net 37 "Net-(J3-Pad26)")
+  (net 38 "Net-(J3-Pad28)")
+  (net 39 "Net-(J3-Pad30)")
+  (net 40 "Net-(J3-Pad34)")
   (net 41 "Net-(KB5-Pad2)")
   (net 42 "Net-(D3-Pad1)")
@@
       (net 4 "+5V") (pinfunction "VCC") (pintype "power_in"))
     (pad "21" thru_hole oval (at 15.24 48.26) (size 1.6 1.6) (drill 0.8) (layers *.Cu *.Mask)
-      (net 37 "Net-(J2-Pad26)") (pinfunction "~{IRQ}") (pintype "output"))
+      (net 37 "Net-(J3-Pad26)") (pinfunction "~{IRQ}") (pintype "output"))
     (pad "22" thru_hole oval (at 15.24 45.72) (size 1.6 1.6) (drill 0.8) (layers *.Cu *.Mask)
-      (net 39 "Net-(J2-Pad30)") (pinfunction "R/~{W}") (pintype "input"))
+      (net 39 "Net-(J3-Pad30)") (pinfunction "R/~{W}") (pintype "input"))
     (pad "23" thru_hole oval (at 15.24 43.18) (size 1.6 1.6) (drill 0.8) (layers *.Cu *.Mask)
       (net 47 "Net-(U2-Pad8)") (pinfunction "~{CS2}") (pintype "input"))
@@
       (net 9 "/A13") (pinfunction "CS1") (pintype "input"))
     (pad "25" thru_hole oval (at 15.24 38.1) (size 1.6 1.6) (drill 0.8) (layers *.Cu *.Mask)
-      (net 38 "Net-(J2-Pad28)") (pinfunction "PHI2") (pintype "input"))
+      (net 38 "Net-(J3-Pad28)") (pinfunction "PHI2") (pintype "input"))
     (pad "26" thru_hole oval (at 15.24 35.56) (size 1.6 1.6) (drill 0.8) (layers *.Cu *.Mask)
       (net 14 "/D7") (pinfunction "D7") (pintype "tri_state"))
@@
     (fp_line (start 8.23 -1.25) (end 1.93 -1.25) (layer "F.Fab") (width 0.1))
     (pad "1" thru_hole circle (at 0 0) (size 1.6 1.6) (drill 0.8) (layers *.Cu *.Mask)
-      (net 40 "Net-(J2-Pad34)") (pintype "passive"))
+      (net 40 "Net-(J3-Pad34)") (pintype "passive"))
     (pad "2" thru_hole oval (at 10.16 0) (size 1.6 1.6) (drill 0.8) (layers *.Cu *.Mask)
       (net 4 "+5V") (pintype "passive"))
@@
       (net 45 "Net-(U2-Pad10)") (pintype "output"))
     (pad "4" thru_hole oval (at 0 7.62) (size 1.6 1.6) (drill 0.8) (layers *.Cu *.Mask)
-      (net 38 "Net-(J2-Pad28)") (pintype "input"))
+      (net 38 "Net-(J3-Pad28)") (pintype "input"))
     (pad "5" thru_hole oval (at 0 10.16) (size 1.6 1.6) (drill 0.8) (layers *.Cu *.Mask)
       (net 45 "Net-(U2-Pad10)") (pintype "input"))
@@
       (net 9 "/A13") (pinfunction "A13") (pintype "input"))
     (pad "27" thru_hole oval (at 15.24 2.54) (size 1.6 1.6) (drill 0.8) (layers *.Cu *.Mask)
-      (net 39 "Net-(J2-Pad30)") (pinfunction "~{WE}") (pintype "input"))
+      (net 39 "Net-(J3-Pad30)") (pinfunction "~{WE}") (pintype "input"))
     (pad "28" thru_hole oval (at 15.24 0) (size 1.6 1.6) (drill 0.8) (layers *.Cu *.Mask)
       (net 4 "+5V") (pinfunction "VCC") (pintype "power_in"))
@@
     (property "Sheetname" "")
     (attr through_hole)
-    (fp_text reference "J2" (at 1.27 -2.33) (layer "F.SilkS")
+    (fp_text reference "J3" (at 1.27 -2.33) (layer "F.SilkS")
       (effects (font (size 1 1) (thickness 0.15)))
     )
@@
       (net 31 "/A8") (pinfunction "Pin_25") (pintype "passive"))
     (pad "26" thru_hole oval (at 2.54 30.48) (size 1.7 1.7) (drill 1) (layers *.Cu *.Mask)
-      (net 37 "Net-(J2-Pad26)") (pinfunction "Pin_26") (pintype "passive"))
+      (net 37 "Net-(J3-Pad26)") (pinfunction "Pin_26") (pintype "passive"))
     (pad "27" thru_hole oval (at 0 33.02) (size 1.7 1.7) (drill 1) (layers *.Cu *.Mask)
       (net 33 "/A9") (pinfunction "Pin_27") (pintype "passive"))
     (pad "28" thru_hole oval (at 2.54 33.02) (size 1.7 1.7) (drill 1) (layers *.Cu *.Mask)
-      (net 38 "Net-(J2-Pad28)") (pinfunction "Pin_28") (pintype "passive"))
+      (net 38 "Net-(J3-Pad28)") (pinfunction "Pin_28") (pintype "passive"))
     (pad "29" thru_hole oval (at 0 35.56) (size 1.7 1.7) (drill 1) (layers *.Cu *.Mask)
       (net 34 "/A10") (pinfunction "Pin_29") (pintype "passive"))
     (pad "30" thru_hole oval (at 2.54 35.56) (size 1.7 1.7) (drill 1) (layers *.Cu *.Mask)
-      (net 39 "Net-(J2-Pad30)") (pinfunction "Pin_30") (pintype "passive"))
+      (net 39 "Net-(J3-Pad30)") (pinfunction "Pin_30") (pintype "passive"))
     (pad "31" thru_hole oval (at 0 38.1) (size 1.7 1.7) (drill 1) (layers *.Cu *.Mask)
       (net 35 "/A11") (pinfunction "Pin_31") (pintype "passive"))
@@
       (net 7 "/A12") (pinfunction "Pin_33") (pintype "passive"))
     (pad "34" thru_hole oval (at 2.54 40.64) (size 1.7 1.7) (drill 1) (layers *.Cu *.Mask)
-      (net 40 "Net-(J2-Pad34)") (pinfunction "Pin_34") (pintype "passive"))
+      (net 40 "Net-(J3-Pad34)") (pinfunction "Pin_34") (pintype "passive"))
     (pad "35" thru_hole oval (at 0 43.18) (size 1.7 1.7) (drill 1) (layers *.Cu *.Mask)
       (net 9 "/A13") (pinfunction "Pin_35") (pintype "passive"))
@@
       (net 1 "GND") (pinfunction "GND") (pintype "power_in"))
     (pad "8" thru_hole circle locked (at 15.24 -7.62 270) (size 1.6 1.6) (drill 0.8) (layers *.Cu *.Mask)
-      (net 38 "Net-(J2-Pad28)") (pinfunction "OUT") (pintype "output"))
+      (net 38 "Net-(J3-Pad28)") (pinfunction "OUT") (pintype "output"))
     (pad "14" thru_hole circle locked (at 0 -7.62 270) (size 1.6 1.6) (drill 0.8) (layers *.Cu *.Mask)
       (net 4 "+5V") (pinfunction "Vcc") (pintype "power_in"))
@@
       (net 49 "unconnected-(U3-Pad3)") (pinfunction "PHI1out") (pintype "output+no_connect"))
     (pad "4" thru_hole oval (at 0 7.62) (size 1.6 1.6) (drill 0.8) (layers *.Cu *.Mask)
-      (net 37 "Net-(J2-Pad26)") (pinfunction "~{IRQ}") (pintype "input"))
+      (net 37 "Net-(J3-Pad26)") (pinfunction "~{IRQ}") (pintype "input"))
     (pad "5" thru_hole oval (at 0 10.16) (size 1.6 1.6) (drill 0.8) (layers *.Cu *.Mask)
       (net 50 "unconnected-(U3-Pad5)") (pinfunction "~{ML}") (pintype "output+no_connect"))
     (pad "6" thru_hole oval (at 0 12.7) (size 1.6 1.6) (drill 0.8) (layers *.Cu *.Mask)
-      (net 40 "Net-(J2-Pad34)") (pinfunction "~{NMI}") (pintype "input"))
+      (net 40 "Net-(J3-Pad34)") (pinfunction "~{NMI}") (pintype "input"))
     (pad "7" thru_hole oval (at 0 15.24) (size 1.6 1.6) (drill 0.8) (layers *.Cu *.Mask)
       (net 51 "unconnected-(U3-Pad7)") (pinfunction "SYNC") (pintype "output+no_connect"))
@@
       (net 26 "/D0") (pinfunction "D0") (pintype "tri_state"))
     (pad "34" thru_hole oval (at 15.24 15.24) (size 1.6 1.6) (drill 0.8) (layers *.Cu *.Mask)
-      (net 39 "Net-(J2-Pad30)") (pinfunction "R/~{W}") (pintype "output"))
+      (net 39 "Net-(J3-Pad30)") (pinfunction "R/~{W}") (pintype "output"))
     (pad "35" thru_hole oval (at 15.24 12.7) (size 1.6 1.6) (drill 0.8) (layers *.Cu *.Mask)
       (net 52 "unconnected-(U3-Pad35)") (pinfunction "NC") (pintype "no_connect"))
@@
       (net 4 "+5V") (pinfunction "BE") (pintype "input"))
     (pad "37" thru_hole oval (at 15.24 7.62) (size 1.6 1.6) (drill 0.8) (layers *.Cu *.Mask)
-      (net 38 "Net-(J2-Pad28)") (pinfunction "PHI2") (pintype "input"))
+      (net 38 "Net-(J3-Pad28)") (pinfunction "PHI2") (pintype "input"))
     (pad "38" thru_hole oval (at 15.24 5.08) (size 1.6 1.6) (drill 0.8) (layers *.Cu *.Mask)
       (net 53 "unconnected-(U3-Pad38)") (pinfunction "~{SO}") (pintype "output+no_connect"))
@@
     (fp_arc (start 63.7 8) (mid 64.053553 8.146447) (end 64.2 8.5) (layer "F.SilkS") (width 0.12))
     (fp_arc (start 0.20066 22.9997) (mid -0.153162 22.853142) (end -0.29972 22.49932) (layer "F.SilkS") (width 0.12))
-    (fp_arc (start 64.20104 22.49932) (mid 64.054479 22.85315) (end 63.70066 22.9997) (layer "F.SilkS") (width 0.12))
+    (fp_arc (start 64.20104 22.49932) (mid 64.054473 22.853115) (end 63.70066 22.9997) (layer "F.SilkS") (width 0.12))
     (fp_line (start -8.25 33.75) (end 72.25 33.75) (layer "F.CrtYd") (width 0.05))
     (fp_line (start 72.25 -2.75) (end 72.25 33.75) (layer "F.CrtYd") (width 0.05))
@@
     (property "Sheetname" "")
     (attr through_hole)
-    (fp_text reference "J1" (at -8.45 5.75 90) (layer "F.SilkS")
+    (fp_text reference "J2" (at -8.45 5.75 90) (layer "F.SilkS")
       (effects (font (size 1 1) (thickness 0.15)))
     )

Commit message: Update windemere-basic.kicad_pcb
Parts:
- moved C10 5.65 mm to (180.4, 122.2)
Routing:
- net GND: track 53.4 -> 93.5 mm
- net +5V: track 533.8 -> 529.3 mm
Changed lines of the file:
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@@
       (effects (font (size 1 1) (thickness 0.15)))
     )
-    (fp_text value "28C256" (at 10 43) (layer "F.Fab")
+    (fp_text value "28C256" (at 11.445 43) (layer "F.Fab")
       (effects (font (size 1 1) (thickness 0.15)))
     )
@@
     (property "Sheetname" "")
     (attr through_hole)
-    (fp_text reference "C11" (at 2.5 -2.5 90) (layer "F.SilkS")
+    (fp_text reference "C11" (at 7.58 0) (layer "F.SilkS")
       (effects (font (size 1 1) (thickness 0.15)))
     )
@@
     (property "Sheetname" "")
     (attr through_hole)
-    (fp_text reference "RV1" (at -2.54 -3.66 90) (layer "F.SilkS")
+    (fp_text reference "RV1" (at 3.8 0) (layer "F.SilkS")
       (effects (font (size 1 1) (thickness 0.15)))
     )
@@
   )
   (footprint "Capacitor_THT:C_Disc_D7.0mm_W2.5mm_P5.00mm" (layer "F.Cu")
-    (at 174.975 120.475)
+    (at 180.365 122.16)
     (descr "C, Disc series, Radial, pin pitch=5.00mm, , diameter*width=7*2.5mm^2, Capacitor, http://cdn-reichelt.de/documents/datenblatt/B300/DS_KERKO_TC.pdf")
     (tags "C Disc series Radial pin pitch 5.00mm  diameter 7mm width 2.5mm Capacitor")
@@
     (property "Sheetname" "")
     (attr through_hole)
-    (fp_text reference "C10" (at 2.5 -2.5) (layer "F.SilkS")
+    (fp_text reference "C10" (at 3.175 -2.54) (layer "F.SilkS")
       (effects (font (size 1 1) (thickness 0.15)))
     )
@@
     (property "Sheetname" "")
     (attr through_hole)
-    (fp_text reference "X1" (at -3.83 -4.4068) (layer "F.SilkS")
+    (fp_text reference "X1" (at -3.755 -6.5424) (layer "F.SilkS")
       (effects (font (size 1 1) (thickness 0.15)))
     )
@@
     (property "Sheetname" "")
     (attr through_hole)
-    (fp_text reference "C5" (at 2.5 2.5) (layer "F.SilkS")
+    (fp_text reference "C5" (at 2.5 0) (layer "F.SilkS")
       (effects (font (size 1 1) (thickness 0.15)))
     )
@@
     (fp_arc (start 63.7 8) (mid 64.053553 8.146447) (end 64.2 8.5) (layer "F.SilkS") (width 0.12))
     (fp_arc (start 0.20066 22.9997) (mid -0.153162 22.853142) (end -0.29972 22.49932) (layer "F.SilkS") (width 0.12))
-    (fp_arc (start 64.20104 22.49932) (mid 64.054473 22.853115) (end 63.70066 22.9997) (layer "F.SilkS") (width 0.12))
+    (fp_arc (start 64.20104 22.49932) (mid 64.054479 22.85315) (end 63.70066 22.9997) (layer "F.SilkS") (width 0.12))
     (fp_line (start -8.25 33.75) (end 72.25 33.75) (layer "F.CrtYd") (width 0.05))
     (fp_line (start 72.25 -2.75) (end 72.25 33.75) (layer "F.CrtYd") (width 0.05))
@@
     (property "Sheetname" "")
     (attr through_hole)
-    (fp_text reference "C2" (at -2 -1.5) (layer "F.SilkS")
+    (fp_text reference "C2" (at -1.45 -2.33) (layer "F.SilkS")
       (effects (font (size 1 1) (thickness 0.15)))
     )
@@
   (segment (start 172.375 167.125) (end 172.375 172.475) (width 0.25) (layer "F.Cu") (net 1))
   (segment (start 167.03 63.105) (end 169.57 65.645) (width 0.25) (layer "F.Cu") (net 1))
+  (segment (start 149.885 160.26) (end 149.870257 160.245257) (width 0.25) (layer "F.Cu") (net 1))
   (segment (start 146.844865 133.720746) (end 147.485465 133.720746) (width 0.25) (layer "F.Cu") (net 1))
   (segment (start 173.875 165.738) (end 173.65 165.962) (width 0.25) (layer "F.Cu") (net 1))
   (segment (start 163.4675 60.475) (end 159.5675 64.375) (width 0.25) (layer "F.Cu") (net 1))
+  (segment (start 161.425654 148.719346) (end 149.885 160.26) (width 0.25) (layer "F.Cu") (net 1))
   (segment (start 153.275 127.931211) (end 153.275 127.875) (width 0.25) (layer "F.Cu") (net 1))
   (segment (start 144.825 135.925) (end 144.825 135.740611) (width 0.25) (layer "F.Cu") (net 1))
@@
   (segment (start 173.65 173.75) (end 173.65 175.85) (width 0.25) (layer "F.Cu") (net 1))
   (segment (start 170.6 178.9) (end 169.07 178.9) (width 0.25) (layer "F.Cu") (net 1))
+  (segment (start 161.425654 143.590257) (end 161.425654 148.719346) (width 0.25) (layer "F.Cu") (net 1))
+  (segment (start 149.870257 160.245257) (end 147.310654 160.245257) (width 0.25) (layer "F.Cu") (net 1))
   (segment (start 173.875 163.625) (end 173.875 165.738) (width 0.25) (layer "F.Cu") (net 1))
   (segment (start 147.485465 133.720746) (end 153.275 127.931211) (width 0.25) (layer "F.Cu") (net 1))
@@
   (segment (start 172.375 172.475) (end 173.65 173.75) (width 0.25) (layer "F.Cu") (net 1))
   (segment (start 173.65 165.962) (end 172.488 167.125) (width 0.25) (layer "F.Cu") (net 1))
+  (segment (start 162.550654 142.465257) (end 161.425654 143.590257) (width 0.25) (layer "F.Cu") (net 1))
   (via (at 173.875 163.625) (size 0.8) (drill 0.4) (layers "F.Cu" "B.Cu") (net 1))
   (via (at 159.41 64.375) (size 0.8) (drill 0.4) (layers "F.Cu" "B.Cu") (net 1))
@@
   (via (at 144.825 135.925) (size 0.8) (drill 0.4) (layers "F.Cu" "B.Cu") (net 1))
   (via (at 169.57 65.645) (size 0.8) (drill 0.4) (layers "F.Cu" "B.Cu") (free) (net 1))
-  (segment (start 141.465 141.735) (end 143.455 143.725) (width 0.25) (layer "B.Cu") (net 1))
+  (segment (start 147.776645 143.590257) (end 143.320257 143.590257) (width 0.25) (layer "B.Cu") (net 1))
+  (segment (start 161.750655 143.265256) (end 148.101646 143.265256) (width 0.25) (layer "B.Cu") (net 1))
   (segment (start 141.465 139.195) (end 141.465 136.655) (width 0.25) (layer "B.Cu") (net 1))
-  (segment (start 143.455 143.725) (end 148.525 143.725) (width 0.25) (layer "B.Cu") (net 1))
+  (segment (start 162.550654 142.465257) (end 161.750655 143.265256) (width 0.25) (layer "B.Cu") (net 1))
+  (segment (start 143.320257 143.590257) (end 141.465 141.735) (width 0.25) (layer "B.Cu") (net 1))
+  (segment (start 148.101646 143.265256) (end 147.776645 143.590257) (width 0.25) (layer "B.Cu") (net 1))
   (segment (start 200.47 189.425) (end 217.755 172.14) (width 0.25) (layer "F.Cu") (net 2))
   (segment (start 160.325 187.575) (end 162.175 189.425) (width 0.25) (layer "F.Cu") (net 2))
@@
   (segment (start 169.07 139.922) (end 169.708 139.285) (width 0.25) (layer "F.Cu") (net 4))
   (segment (start 164.249 166.2) (end 163.124 167.325) (width 0.25) (layer "B.Cu") (net 4))
-  (segment (start 184.49 128) (end 175.115 118.625) (width 0.25) (layer "B.Cu") (net 4))
   (segment (start 162.455 79.325) (end 161.33 79.325) (width 0.25) (layer "B.Cu") (net 4))
   (segment (start 183.817 170.099) (end 184.942 171.224) (width 0.25) (layer "B.Cu") (net 4))
   (segment (start 160.325 168.198) (end 160.325 169.83) (width 0.25) (layer "B.Cu") (net 4))
-  (segment (start 170.815 118.625) (end 170.75 118.56) (width 0.25) (layer "B.Cu") (net 4))
   (segment (start 153.71 86.945) (end 147.215 86.945) (width 0.25) (layer "B.Cu") (net 4))
   (segment (start 257.986 79.2089) (end 239.929 79.2089) (width 0.25) (layer "B.Cu") (net 4))
+  (segment (start 170.815 118.625) (end 170.75 118.56) (width 0.25) (layer "B.Cu") (net 4))
   (segment (start 217.099 79.221) (end 199.416 79.221) (width 0.25) (layer "B.Cu") (net 4))
   (segment (start 178.38 38.625) (end 179.505 38.625) (width 0.25) (layer "B.Cu") (net 4))
@@
   (segment (start 165.3533 48.425) (end 168.22 45.5583) (width 0.25) (layer "B.Cu") (net 4))
   (segment (start 165.4747 127.2253) (end 167.699511 125.000489) (width 0.25) (layer "B.Cu") (net 4))
+  (segment (start 176.83 118.625) (end 170.815 118.625) (width 0.25) (layer "B.Cu") (net 4))
   (segment (start 170.75 117.435) (end 170.75 118.56) (width 0.25) (layer "B.Cu") (net 4))
   (segment (start 163.124 167.325) (end 161.197 167.325) (width 0.25) (layer "B.Cu") (net 4))
   (segment (start 161.197 167.325) (end 160.325 168.198) (width 0.25) (layer "B.Cu") (net 4))
+  (segment (start 185.615 127.41) (end 176.83 118.625) (width 0.25) (layer "B.Cu") (net 4))
   (segment (start 259.12 78.075) (end 257.986 79.2089) (width 0.25) (layer "B.Cu") (net 4))
   (segment (start 169.07 166.2) (end 164.249 166.2) (width 0.25) (layer "B.Cu") (net 4))
@@
   (segment (start 220.213 76.1072) (end 220.213 53.2935) (width 0.25) (layer "B.Cu") (net 4))
   (segment (start 218.245 78.075) (end 217.099 79.221) (width 0.25) (layer "B.Cu") (net 4))
-  (segment (start 172.665 120.475) (end 170.815 118.625) (width 0.25) (layer "B.Cu") (net 4))
   (segment (start 156.678 169.83) (end 160.325 169.83) (width 0.25) (layer "B.Cu") (net 4))
   (segment (start 151.2325 56.78) (end 152.511 56.78) (width 0.25) (layer "B.Cu") (net 4))
@@
   (segment (start 204.553 39.9425) (end 204.17 39.9425) (width 0.25) (layer "B.Cu") (net 4))
   (segment (start 236.827 76.1072) (end 220.213 76.1072) (width 0.25) (layer "B.Cu") (net 4))
+  (segment (start 185.615 128) (end 185.615 127.41) (width 0.25) (layer "B.Cu") (net 4))
   (segment (start 236.807 39.9425) (end 237.19 39.9425) (width 0.25) (layer "B.Cu") (net 4))
   (segment (start 220.213 53.2935) (end 223.456 53.2935) (width 0.25) (layer "B.Cu") (net 4))
   (segment (start 152.511 56.78) (end 160.866 48.425) (width 0.25) (layer "B.Cu") (net 4))
   (segment (start 238.795 78.075) (end 236.827 76.1072) (width 0.25) (layer "B.Cu") (net 4))
-  (segment (start 175.115 118.625) (end 170.815 118.625) (width 0.25) (layer "B.Cu") (net 4))
   (segment (start 167.699511 125.000489) (end 167.699511 121.610489) (width 0.25) (layer "B.Cu") (net 4))
   (segment (start 162.5507 127.2253) (end 165.4747 127.2253) (width 0.25) (layer "B.Cu") (net 4))
-  (segment (start 185.615 128) (end 184.49 128) (width 0.25) (layer "B.Cu") (net 4))
   (segment (start 203.964 38.1109) (end 204.17 38.3172) (width 0.25) (layer "B.Cu") (net 4))
   (segment (start 179.505 38.625) (end 180.019 38.1109) (width 0.25) (layer "B.Cu") (net 4))
@@
   (segment (start 174.514 170.099) (end 183.817 170.099) (width 0.25) (layer "B.Cu") (net 4))
   (segment (start 220.213 53.2935) (end 217.904 53.2935) (width 0.25) (layer "B.Cu") (net 4))
-  (segment (start 174.975 120.475) (end 172.665 120.475) (width 0.25) (layer "B.Cu") (net 4))
   (segment (start 186.08 56.13) (end 190.5225 56.13) (width 0.25) (layer "F.Cu") (net 6))
   (segment (start 190.5225 56.13) (end 206.71 39.9425) (width 0.25) (layer "F.Cu") (net 6))

Commit message: Cleanup the Schematic
Changed lines of the file:
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@@
     (fp_arc (start 63.7 8) (mid 64.053553 8.146447) (end 64.2 8.5) (layer "F.SilkS") (width 0.12))
     (fp_arc (start 0.20066 22.9997) (mid -0.153162 22.853142) (end -0.29972 22.49932) (layer "F.SilkS") (width 0.12))
-    (fp_arc (start 64.20104 22.49932) (mid 64.054479 22.85315) (end 63.70066 22.9997) (layer "F.SilkS") (width 0.12))
+    (fp_arc (start 64.20104 22.49932) (mid 64.054473 22.853115) (end 63.70066 22.9997) (layer "F.SilkS") (width 0.12))
     (fp_line (start -8.25 33.75) (end 72.25 33.75) (layer "F.CrtYd") (width 0.05))
     (fp_line (start 72.25 -2.75) (end 72.25 33.75) (layer "F.CrtYd") (width 0.05))
